File: YM2612/Ym2612.sch (EAGLE design)
At the start: 31 parts, among them IC2 74LS14N, IC4 74LS138N, U1 ATMEGA1284P-PU, U2 YM2612_1, U3 YM2612_2, U4 YM2612_2, Y1 16MHz

Commit message: Lots of work
Parts:
- added C15, C5: 22pF, rcl:C-EU050-024X044
- added C16: 0.1uF, rcl:CPOL-EUE2.5-6
- added IC1, IC3: 7805TV, linear:7805TV
- added U5: ATMEGA1284P-PU, ATMEGA1284P-PU:ATMEGA1284P-PU
- added Y2: 16MHz, SparkFun-Clocks:CRYSTAL-16MHZPTH-HC49US
Connections:
- new net +12V: IC1.VI, IC3.VI
- new net 1284_2_XTAL_1: C5.1, U5.XTAL1, Y2.1
- new net 1284_2_XTAL_2: C15.1, U5.XTAL2, Y2.2
- new net A.GND: IC1.GND, IC3.GND
- new net A.VCC: IC3.VO
- net +5V: now also C16.+, IC1.VO, U5.AVCC, U5.VCC
- net 1284_1_RX_1: now also U5.PD1
- net 1284_1_TX_1: now also U5.PD0
- net GND: now also C15.2, C16.-, C5.2, U5.GND, U5.GND_2
